Commit message: description macro

File: MiniProsjekt/qube_description/urdf/cube.urdf.xacro (robot description, xacro)
@@ -1 +1,11 @@
-# scene-fil
+<?xml version="1.0"?>
+<robot xmlns:xacro="http://www.ros.org/wiki/xacro" name="qube_scene">
+  <xacro:include filename="$(find qube_description)/urdf/qube.macro.xacro" />
+  <link name="world"/>
+  <xacro:qube/>
+  <joint name="world_to_base" type="fixed">
+    <parent link="world"/>
+    <child link="base_link"/>
+    <origin xyz="0 0 0" rpy="0 0 0"/>
+  </joint>
+</robot>
