Commit message: description all

File: MiniProsjekt/qube_description/urdf/cube.macro.xacro (robot description, xacro)
@@ -1,10 +1,18 @@
 <?xml version="1.0"?>
 <robot xmlns:xacro="http://www.ros.org/wiki/xacro">
-  <xacro:macro name="qube" params="length:=0.1 width:=0.1 height:=0.1 disk_radius:=0.05 disk_thickness:=0.01">
-    <!-- Description of qube -->
+  <!-- Macro-parametre -->
+  <xacro:property name="base_length" value="0.1" />
+  <xacro:property name="base_width" value="0.1" />
+  <xacro:property name="base_height" value="0.1" />
+  <xacro:property name="disk_radius" value="0.05" />
+  <xacro:property name="disk_height" value="0.02" />
+  <xacro:property name="pointer_length" value="0.04" />
+  <xacro:property name="pointer_radius" value="0.005" />
+  <xacro:macro name="qube">
+    <!-- Base -->
     <link name="base_link">
       <visual>
         <geometry>
-          <box size="${length} ${width} ${height}"/>
+          <box size="${base_length} ${base_width} ${base_height}"/>
         </geometry>
         <material name="black">
@@ -12,14 +20,10 @@
         </material>
       </visual>
-      <collision>
-        <geometry>
-          <box size="${length} ${width} ${height}"/>
-        </geometry>
-      </collision>
     </link>
-    <link name="disk">
+    <!-- Roterende disk -->
+    <link name="rotating_disk">
       <visual>
         <geometry>
-          <cylinder radius="${disk_radius}" length="${disk_thickness}"/>
+          <cylinder radius="${disk_radius}" length="${disk_height}"/>
         </geometry>
         <material name="red">
@@ -27,20 +31,16 @@
         </material>
       </visual>
-      <collision>
-        <geometry>
-          <cylinder radius="${disk_radius}" length="${disk_thickness}"/>
-        </geometry>
-      </collision>
     </link>
-    <joint name="base_to_disk" type="continuous">
+    <joint name="disk_joint" type="continuous">
       <parent link="base_link"/>
-      <child link="disk"/>
-      <origin xyz="0 0 ${height/2 + disk_thickness/2}" rpy="0 0 0"/>
+      <child link="rotating_disk"/>
+      <origin xyz="0 0 ${base_height/2 + disk_height/2}"/>
       <axis xyz="0 0 1"/>
     </joint>
-    <link name="indicator">
+    <!-- Hvit viser -->
+    <link name="pointer">
       <visual>
         <geometry>
-          <box size="${disk_radius*0.8} ${disk_thickness} ${disk_thickness}"/>
+          <cylinder radius="${pointer_radius}" length="${pointer_length}"/>
         </geometry>
         <material name="white">
@@ -49,10 +49,9 @@
       </visual>
     </link>
-    <joint name="disk_to_indicator" type="fixed">
-      <parent link="disk"/>
-      <child link="indicator"/>
-      <origin xyz="${disk_radius*0.4} 0 ${disk_thickness/2}" rpy="0 0 0"/>
+    <joint name="pointer_joint" type="fixed">
+      <parent link="rotating_disk"/>
+      <child link="pointer"/>
+      <origin xyz="${disk_radius - pointer_length/2} 0 0"/>
     </joint>
-    <!-- End of Description -->
   </xacro:macro>
 </robot>

File: MiniProsjekt/qube_description/urdf/cube.urdf.xacro (robot description, xacro)
@@ -1,11 +1,14 @@
 <?xml version="1.0"?>
-<robot xmlns:xacro="http://www.ros.org/wiki/xacro" name="qube_scene">
+<robot xmlns:xacro="http://www.ros.org/wiki/xacro">
   <xacro:include filename="$(find qube_description)/urdf/qube.macro.xacro" />
+  <!-- World link -->
   <link name="world"/>
+  <!-- Instansier Qube-makro -->
   <xacro:qube/>
-  <joint name="world_to_base" type="fixed">
+  <!-- Fest base_link til world -->
+  <joint name="world_base_joint" type="fixed">
     <parent link="world"/>
     <child link="base_link"/>
-    <origin xyz="0 0 0" rpy="0 0 0"/>
+    <origin xyz="0 0 0"/>
   </joint>
 </robot>
