Commit message: Fix Lab3

File: src/joint_description/urdf/joint_model.urdf (robot description, URDF)
Before this commit: robot joint_model, 5 links, 4 joints
Links:
- removed link angle_link
- removed link rotor_link
- removed link stator_link
Joints:
- removed joint angle
- removed joint indicator
