Commit message: mye fiks..

File: MiniProsjekt/src/qube_description/urdf/qube.macro.xacro (robot description, xacro)
@@ -2,15 +2,20 @@
 <robot xmlns:xacro="http://www.ros.org/wiki/xacro">
   <!-- Macro-parametre -->
-  <xacro:property name="base_length" value="0.1" />
-  <xacro:property name="base_width" value="0.1" />
-  <xacro:property name="base_height" value="0.1" />
-  <xacro:property name="disk_radius" value="0.05" />
-  <xacro:property name="disk_height" value="0.02" />
-  <xacro:property name="pointer_length" value="0.04" />
-  <xacro:property name="pointer_radius" value="0.005" />
+  <xacro:property name="base_length" value="1" />
+  <xacro:property name="base_width" value="1" />
+  <xacro:property name="base_height" value="1" />
+  <xacro:property name="disk_radius" value="0.5" />
+  <xacro:property name="disk_height" value="0.2" />
+  <xacro:property name="pointer_length" value="0.4" />
+  <xacro:property name="pointer_radius" value="0.05" />
   <xacro:macro name="qube">
     <!-- Base -->
     <link name="base_link">
+      <inertial>
+        <mass value="1" />
+        <inertia ixx="0.1" iyy="0.1" izz="0.1" ixy="0" ixz="0" iyz="0" />
+      </inertial>
       <visual>
+        <origin xyz="0 0 0" rpy="0 0 0"/>
         <geometry>
           <box size="${base_length} ${base_width} ${base_height}"/>
@@ -23,5 +28,10 @@
     <!-- Roterende disk -->
     <link name="rotating_disk">
+      <inertial>
+        <mass value="0.5" />
+        <inertia ixx="0.05" iyy="0.05" izz="0.05" ixy="0" ixz="0" iyz="0" />
+      </inertial>
       <visual>
+        <origin xyz="0 0 0" rpy="0 0 0"/>
         <geometry>
           <cylinder radius="${disk_radius}" length="${disk_height}"/>
@@ -40,5 +50,10 @@
     <!-- Hvit viser -->
     <link name="pointer">
+      <inertial>
+        <mass value="0.1" />
+        <inertia ixx="0.01" iyy="0.01" izz="0.01" ixy="0" ixz="0" iyz="0" />
+      </inertial>
       <visual>
+        <origin xyz="0 0 0" rpy="0 0 0"/>
         <geometry>
           <cylinder radius="${pointer_radius}" length="${pointer_length}"/>

File: MiniProsjekt/src/qube_description/urdf/qube.urdf.xacro (robot description, xacro)
@@ -1,4 +1,4 @@
 <?xml version="1.0"?>
-<robot xmlns:xacro="http://www.ros.org/wiki/xacro">
+<robot name="qube_robot" xmlns:xacro="http://www.ros.org/wiki/xacro">
   <xacro:include filename="$(find qube_description)/urdf/qube.macro.xacro" />
   <!-- World link -->

Commit message: ugh

File: MiniProsjekt/src/qube_description/urdf/qube.macro.xacro (robot description, xacro)
@@ -12,10 +12,5 @@
     <!-- Base -->
     <link name="base_link">
-      <inertial>
-        <mass value="1" />
-        <inertia ixx="0.1" iyy="0.1" izz="0.1" ixy="0" ixz="0" iyz="0" />
-      </inertial>
       <visual>
-        <origin xyz="0 0 0" rpy="0 0 0"/>
         <geometry>
           <box size="${base_length} ${base_width} ${base_height}"/>
@@ -25,13 +20,13 @@
         </material>
       </visual>
+      <inertial>
+        <mass value="1.0"/>
+        <origin xyz="0 0 0"/>
+        <inertia ixx="0.1" ixy="0.0" ixz="0.0" iyy="0.1" iyz="0.0" izz="0.1"/>
+      </inertial>
     </link>
     <!-- Roterende disk -->
     <link name="rotating_disk">
-      <inertial>
-        <mass value="0.5" />
-        <inertia ixx="0.05" iyy="0.05" izz="0.05" ixy="0" ixz="0" iyz="0" />
-      </inertial>
       <visual>
-        <origin xyz="0 0 0" rpy="0 0 0"/>
         <geometry>
           <cylinder radius="${disk_radius}" length="${disk_height}"/>
@@ -41,4 +36,9 @@
         </material>
       </visual>
+      <inertial>
+        <mass value="0.5"/>
+        <origin xyz="0 0 0"/>
+        <inertia ixx="0.05" ixy="0.0" ixz="0.0" iyy="0.05" iyz="0.0" izz="0.05"/>
+      </inertial>
     </link>
     <joint name="disk_joint" type="continuous">
@@ -50,10 +50,5 @@
     <!-- Hvit viser -->
     <link name="pointer">
-      <inertial>
-        <mass value="0.1" />
-        <inertia ixx="0.01" iyy="0.01" izz="0.01" ixy="0" ixz="0" iyz="0" />
-      </inertial>
       <visual>
-        <origin xyz="0 0 0" rpy="0 0 0"/>
         <geometry>
           <cylinder radius="${pointer_radius}" length="${pointer_length}"/>
@@ -63,4 +58,9 @@
         </material>
       </visual>
+      <inertial>
+        <mass value="0.1"/>
+        <origin xyz="0 0 0"/>
+        <inertia ixx="0.01" ixy="0.0" ixz="0.0" iyy="0.01" iyz="0.0" izz="0.01"/>
+      </inertial>
     </link>
     <joint name="pointer_joint" type="fixed">

Commit message: RViz funker

File: MiniProsjekt/src/qube_description/urdf/qube.macro.xacro (robot description, xacro)
@@ -1,5 +1,15 @@
 <?xml version="1.0"?>
-<robot xmlns:xacro="http://www.ros.org/wiki/xacro">
-  <!-- Macro-parametre -->
+<robot name="qube_robot" xmlns:xacro="http://www.ros.org/wiki/xacro">
+  <!-- Globale materialer -->
+  <material name="black">
+    <color rgba="0 0 0 1"/>
+  </material>
+  <material name="red">
+    <color rgba="1 0 0 1"/>
+  </material>
+  <material name="white">
+    <color rgba="1 1 1 1"/>
+  </material>
+  <!-- Makro-parametre -->
   <xacro:property name="base_length" value="1" />
   <xacro:property name="base_width" value="1" />
@@ -13,15 +23,14 @@
     <link name="base_link">
       <visual>
+        <origin xyz="0 0 0" rpy="0 0 0"/>
         <geometry>
           <box size="${base_length} ${base_width} ${base_height}"/>
         </geometry>
-        <material name="black">
-          <color rgba="0 0 0 1"/>
-        </material>
+        <material name="black"/>
       </visual>
       <inertial>
         <mass value="1.0"/>
         <origin xyz="0 0 0"/>
-        <inertia ixx="0.1" ixy="0.0" ixz="0.0" iyy="0.1" iyz="0.0" izz="0.1"/>
+        <inertia ixx="0.1" ixy="0" ixz="0" iyy="0.1" iyz="0" izz="0.1"/>
       </inertial>
     </link>
@@ -29,15 +38,14 @@
     <link name="rotating_disk">
       <visual>
+        <origin xyz="0 0 0" rpy="0 0 0"/>
         <geometry>
           <cylinder radius="${disk_radius}" length="${disk_height}"/>
         </geometry>
-        <material name="red">
-          <color rgba="1 0 0 1"/>
-        </material>
+        <material name="red"/>
       </visual>
       <inertial>
         <mass value="0.5"/>
         <origin xyz="0 0 0"/>
-        <inertia ixx="0.05" ixy="0.0" ixz="0.0" iyy="0.05" iyz="0.0" izz="0.05"/>
+        <inertia ixx="0.05" ixy="0" ixz="0" iyy="0.05" iyz="0" izz="0.05"/>
       </inertial>
     </link>
@@ -51,15 +59,14 @@
     <link name="pointer">
       <visual>
+        <origin xyz="0 0 0" rpy="0 1.5708 0"/> <!-- Roter 90° om Y-aksen -->
         <geometry>
           <cylinder radius="${pointer_radius}" length="${pointer_length}"/>
         </geometry>
-        <material name="white">
-          <color rgba="1 1 1 1"/>
-        </material>
+        <material name="white"/>
       </visual>
       <inertial>
         <mass value="0.1"/>
         <origin xyz="0 0 0"/>
-        <inertia ixx="0.01" ixy="0.0" ixz="0.0" iyy="0.01" iyz="0.0" izz="0.01"/>
+        <inertia ixx="0.01" ixy="0" ixz="0" iyy="0.01" iyz="0" izz="0.01"/>
       </inertial>
     </link>
@@ -67,5 +74,5 @@
       <parent link="rotating_disk"/>
       <child link="pointer"/>
-      <origin xyz="${disk_radius - pointer_length/2} 0 0"/>
+      <origin xyz="${disk_radius} 0 0"/> <!-- Plasser ytterkant av disk -->
     </joint>
   </xacro:macro>

Commit message: kommentarer

File: MiniProsjekt/src/qube_description/urdf/qube.macro.xacro (robot description, xacro)
@@ -1,15 +1,5 @@
 <?xml version="1.0"?>
-<robot name="qube_robot" xmlns:xacro="http://www.ros.org/wiki/xacro">
-  <!-- Globale materialer -->
-  <material name="black">
-    <color rgba="0 0 0 1"/>
-  </material>
-  <material name="red">
-    <color rgba="1 0 0 1"/>
-  </material>
-  <material name="white">
-    <color rgba="1 1 1 1"/>
-  </material>
-  <!-- Makro-parametre -->
+<robot xmlns:xacro="http://www.ros.org/wiki/xacro">
+  <!-- Macro-parametre -->
   <xacro:property name="base_length" value="1" />
   <xacro:property name="base_width" value="1" />
@@ -23,14 +13,15 @@
     <link name="base_link">
       <visual>
-        <origin xyz="0 0 0" rpy="0 0 0"/>
         <geometry>
           <box size="${base_length} ${base_width} ${base_height}"/>
         </geometry>
-        <material name="black"/>
+        <material name="black">
+          <color rgba="0 0 0 1"/>
+        </material>
       </visual>
       <inertial>
         <mass value="1.0"/>
         <origin xyz="0 0 0"/>
-        <inertia ixx="0.1" ixy="0" ixz="0" iyy="0.1" iyz="0" izz="0.1"/>
+        <inertia ixx="0.1" ixy="0.0" ixz="0.0" iyy="0.1" iyz="0.0" izz="0.1"/>
       </inertial>
     </link>
@@ -38,14 +29,15 @@
     <link name="rotating_disk">
       <visual>
-        <origin xyz="0 0 0" rpy="0 0 0"/>
         <geometry>
           <cylinder radius="${disk_radius}" length="${disk_height}"/>
         </geometry>
-        <material name="red"/>
+        <material name="red">
+          <color rgba="1 0 0 1"/>
+        </material>
       </visual>
       <inertial>
         <mass value="0.5"/>
         <origin xyz="0 0 0"/>
-        <inertia ixx="0.05" ixy="0" ixz="0" iyy="0.05" iyz="0" izz="0.05"/>
+        <inertia ixx="0.05" ixy="0.0" ixz="0.0" iyy="0.05" iyz="0.0" izz="0.05"/>
       </inertial>
     </link>
@@ -59,14 +51,15 @@
     <link name="pointer">
       <visual>
-        <origin xyz="0 0 0" rpy="0 1.5708 0"/> <!-- Roter 90° om Y-aksen -->
         <geometry>
           <cylinder radius="${pointer_radius}" length="${pointer_length}"/>
         </geometry>
-        <material name="white"/>
+        <material name="white">
+          <color rgba="1 1 1 1"/>
+        </material>
       </visual>
       <inertial>
         <mass value="0.1"/>
         <origin xyz="0 0 0"/>
-        <inertia ixx="0.01" ixy="0" ixz="0" iyy="0.01" iyz="0" izz="0.01"/>
+        <inertia ixx="0.01" ixy="0.0" ixz="0.0" iyy="0.01" iyz="0.0" izz="0.01"/>
       </inertial>
     </link>
@@ -74,5 +67,5 @@
       <parent link="rotating_disk"/>
       <child link="pointer"/>
-      <origin xyz="${disk_radius} 0 0"/> <!-- Plasser ytterkant av disk -->
+      <origin xyz="${disk_radius - pointer_length/2} 0 0"/>
     </joint>
   </xacro:macro>

Commit message: fiksa macro til riktig verdier

File: MiniProsjekt/src/qube_description/urdf/qube.macro.xacro (robot description, xacro)
@@ -12,67 +12,53 @@
   </material>
   <!-- Makro-parametre -->
-  <xacro:property name="base_length" value="1" />
-  <xacro:property name="base_width" value="1" />
-  <xacro:property name="base_height" value="1" />
-  <xacro:property name="disk_radius" value="0.5" />
-  <xacro:property name="disk_height" value="0.2" />
-  <xacro:property name="pointer_length" value="0.4" />
-  <xacro:property name="pointer_radius" value="0.05" />
+  <xacro:property name="base_length" value="0.102" />
+  <xacro:property name="disk_radius" value="0.025" />
+  <xacro:property name="disk_height" value="0.01" />
+  <xacro:property name="pointer_length" value="0.025" />
+  <xacro:property name="pointer_height" value="0.02" />
   <xacro:macro name="qube">
-    <!-- Base -->
+    <!-- Base link og joint -->
     <link name="base_link">
       <visual>
-        <origin xyz="0 0 0" rpy="0 0 0"/>
         <geometry>
-          <box size="${base_length} ${base_width} ${base_height}"/>
+          <box size="${base_length} ${base_length} ${base_length}"/>
         </geometry>
         <material name="black"/>
       </visual>
-      <inertial>
-        <mass value="1.0"/>
-        <origin xyz="0 0 0"/>
-        <inertia ixx="0.1" ixy="0" ixz="0" iyy="0.1" iyz="0" izz="0.1"/>
-      </inertial>
     </link>
-    <!-- Roterende disk -->
+    <joint name="base_joint" type="fixed">
+      <parent link="base_link"/>
+      <child link="rotating_disk"/>
+      <origin xyz="0 0 0.051" rpy="0 0 0"/>
+    </joint>
+    <!-- Roterende disk link og joint -->
     <link name="rotating_disk">
-      <visual>
-        <origin xyz="0 0 0" rpy="0 0 0"/>
-        <geometry>
-          <cylinder radius="${disk_radius}" length="${disk_height}"/>
-        </geometry>
-        <material name="red"/>
-      </visual>
-      <inertial>
-        <mass value="0.5"/>
-        <origin xyz="0 0 0"/>
-        <inertia ixx="0.05" ixy="0" ixz="0" iyy="0.05" iyz="0" izz="0.05"/>
-      </inertial>
+        <visual>
+            <geometry>
+                <cylinder radius="0.025" length="0.01"/>
+            </geometry>
+            <material name="red"/>
+        </visual>
     </link>
     <joint name="disk_joint" type="continuous">
       <parent link="base_link"/>
       <child link="rotating_disk"/>
-      <origin xyz="0 0 ${base_height/2 + disk_height/2}"/>
+      <origin xyz="0 0 0.056" rpy="0 0 0"/>
       <axis xyz="0 0 1"/>
+      <limit lower="-3.14" upper="3.14" effort="10" velocity="5"/>
     </joint>
-    <!-- Hvit viser -->
+    <!-- Hvit viser link og joint -->
     <link name="pointer">
-      <visual>
-        <origin xyz="0 0 0" rpy="0 1.5708 0"/> <!-- Roter 90° om Y-aksen -->
-        <geometry>
-          <cylinder radius="${pointer_radius}" length="${pointer_length}"/>
-        </geometry>
-        <material name="white"/>
-      </visual>
-      <inertial>
-        <mass value="0.1"/>
-        <origin xyz="0 0 0"/>
-        <inertia ixx="0.01" ixy="0" ixz="0" iyy="0.01" iyz="0" izz="0.01"/>
-      </inertial>
+        <visual>
+            <geometry>
+                <box size="0.025 0.002 0.002"/>
+            </geometry>
+            <material name="white"/>
+        </visual>
     </link>
     <joint name="pointer_joint" type="fixed">
       <parent link="rotating_disk"/>
       <child link="pointer"/>
-      <origin xyz="${disk_radius} 0 0"/> <!-- Plasser ytterkant av disk -->
+      <origin xyz="0.0125 0 0.006" rpy="0 0 0"/>
     </joint>
   </xacro:macro>

Commit message: disk_joint to motor_joint

File: MiniProsjekt/src/qube_description/urdf/qube.macro.xacro (robot description, xacro)
@@ -41,5 +41,5 @@
         </visual>
     </link>
-    <joint name="disk_joint" type="continuous">
+    <joint name="motor_joint" type="continuous">
       <parent link="base_link"/>
       <child link="rotating_disk"/>
